File: tb.kicad_sch (KiCad schematic)
At the start: 67 parts, among them U4 JHL6340SLLSQ, U5 MX25L8006EM1I-12G, U6 SI52112-B6-GT, U7 MX25L8006EM2I-12G, Y1 ABM8G-25.000MHZ-B4Y-T, Y2 ABM8G-25.000MHZ-B4Y-T

Commit message: Generate library of local components
Parts:
- C100, C102, C103, C105, C106, C107, C108, C109, C110, C111, C112, C99: footprint antmicro-footprints:C_0402_1005Metric -> thunderbolt-pcie-adapter-footprints:C_0402_1005Metric; symbol antmicroCapacitors0402:C_220n_0402 -> thunderbolt-pcie-adapter:C_220n_0402
- C101, C104, C115, C98: footprint antmicro-footprints:C_0402_1005Metric -> thunderbolt-pcie-adapter-footprints:C_0402_1005Metric; symbol antmicroCapacitors0402:C_100n_0402 -> thunderbolt-pcie-adapter:C_100n_0402
- C113, C114, C116, C117: footprint antmicro-footprints:C_0402_1005Metric -> thunderbolt-pcie-adapter-footprints:C_0402_1005Metric; symbol antmicroCapacitors0402:C_10p_0402 -> thunderbolt-pcie-adapter:C_10p_0402
- R50, R51, R52, R53: footprint antmicro-footprints:R_0402_1005Metric -> thunderbolt-pcie-adapter-footprints:R_0402_1005Metric; symbol antmicroResistors0402:R_3k3_0402 -> thunderbolt-pcie-adapter:R_3k3_0402
- R54, R55, R70, R71, R82: footprint antmicro-footprints:R_0402_1005Metric -> thunderbolt-pcie-adapter-footprints:R_0402_1005Metric; symbol antmicroResistors0402:R_1M_0402 -> thunderbolt-pcie-adapter:R_1M_0402
- R56, R64, R65, R66, R67, R78, R79, R80, R83, R85: footprint antmicro-footprints:R_0402_1005Metric -> thunderbolt-pcie-adapter-footprints:R_0402_1005Metric; symbol antmicroResistors0402:R_10k_0402 -> thunderbolt-pcie-adapter:R_10k_0402
- R57, R60, R72, R75, R77, R81, R84, R86, R87, R90: footprint antmicro-footprints:R_0402_1005Metric -> thunderbolt-pcie-adapter-footprints:R_0402_1005Metric; symbol antmicroResistors0402:R_100k_0402 -> thunderbolt-pcie-adapter:R_100k_0402
- R58, R59, R61, R62: footprint antmicro-footprints:R_0402_1005Metric -> thunderbolt-pcie-adapter-footprints:R_0402_1005Metric; symbol antmicroResistors0402:R_2k2_0402 -> thunderbolt-pcie-adapter:R_2k2_0402
- R63, R76: footprint antmicro-footprints:R_0402_1005Metric -> thunderbolt-pcie-adapter-footprints:R_0402_1005Metric; symbol antmicroResistors0402:R_14k_0402 -> thunderbolt-pcie-adapter:R_14k_0402
- R68, R73: footprint antmicro-footprints:R_0402_1005Metric -> thunderbolt-pcie-adapter-footprints:R_0402_1005Metric; symbol antmicroResistors0402:R_499R_0402 -> thunderbolt-pcie-adapter:R_499R_0402
- R69: footprint antmicro-footprints:R_0402_1005Metric -> thunderbolt-pcie-adapter-footprints:R_0402_1005Metric; symbol antmicroResistors0402:R_4k75_0.5%_0402 -> thunderbolt-pcie-adapter:R_4k75_0.5%_0402
- R74: footprint antmicro-footprints:R_0402_1005Metric -> thunderbolt-pcie-adapter-footprints:R_0402_1005Metric; symbol antmicroResistors0402:R_3k01_0402 -> thunderbolt-pcie-adapter:R_3k01_0402
- R88, R89: footprint antmicro-footprints:R_0402_1005Metric -> thunderbolt-pcie-adapter-footprints:R_0402_1005Metric; symbol antmicroResistors0402:R_100R_0402 -> thunderbolt-pcie-adapter:R_100R_0402
- U4: footprint antmicro-footprints:JHL6340SLLSQ -> thunderbolt-pcie-adapter-footprints:JHL6340SLLSQ; symbol antmicroInterfaceControllers:JHL6340SLLSQ -> thunderbolt-pcie-adapter:JHL6340SLLSQ
- U5: footprint antmicro-footprints:SOIC-8_3.9x4.9x1.75mm_P1.27mm -> thunderbolt-pcie-adapter-footprints:SOIC-8_3.9x4.9x1.75mm_P1.27mm; symbol antmicroMemory:MX25L8006EM1I-12G -> thunderbolt-pcie-adapter:MX25L8006EM1I-12G
- U6: footprint antmicro-footprints:TSSOP-8_3x4.4mm_P0.65mm -> thunderbolt-pcie-adapter-footprints:TSSOP-8_3x4.4mm_P0.65mm; symbol antmicroClockTimingClockGeneratorsPLLsFrequencySynthesizers:SI52112-B6-GT -> thunderbolt-pcie-adapter:SI52112-B6-GT
- U7: footprint antmicro-footprints:SOIC-8_5.3x5.3x2mm_P1.27mm -> thunderbolt-pcie-adapter-footprints:SOIC-8_5.3x5.3x2mm_P1.27mm; symbol antmicroMemory:MX25L8006EM2I-12G -> thunderbolt-pcie-adapter:MX25L8006EM2I-12G
- Y1, Y2: footprint antmicro-footprints:Oscillator_SMD_Geyer_KX-7-4Pin_3.2x2.5mm -> thunderbolt-pcie-adapter-footprints:Oscillator_SMD_Geyer_KX-7-4Pin_3.2x2.5mm; symbol antmicroCrystals:ABM8G-25.000MHZ-B4Y-T -> thunderbolt-pcie-adapter:ABM8G-25.000MHZ-B4Y-T
