File: connectors.kicad_sch (KiCad schematic)
At the start: 13 parts, among them J1 USB-C_JAE_DX07S024JJ2, J2 PCIe_x4_Conn_EdgeMount_Open, J3 Molex_Nano-Fit_1x2_1053131102

Commit message: [#61922] Update all symbols, clean ERC
Parts:
- C1, C2, C3, C4, C5, C6, MP1, MP2, MP3, R1: Public (none) -> False
Changed lines of the file:
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@@
     )
     (property "Value" "MP_Pad6mm_Drill3mm" (at 40.64 265.43 0)
-      (effects (font (size 1.27 1.27) (thickness 0.15)) (justify left) hide)
+      (effects (font (size 1.27 1.27) (thickness 0.15)) (justify left))
     )
     (property "Footprint" "antmicro-footprints:MP_Pad6mm_Drill3mm" (at 52.07 271.78 0)
@@
     (property "License" "Apache-2.0" (at 52.07 276.86 0)
       (effects (font (size 1.27 1.27) (thickness 0.15)) (justify left bottom) hide)
+    )
+    (property "Public" "False" (at 52.07 279.4 0)
+      (effects (font (size 1.27 1.27)) (justify left bottom) hide)
     )
     (pin "1")
@@
     (property "Author" "Antmicro" (at 369.57 85.09 0)
       (effects (font (size 1.27 1.27) (thickness 0.15)) (justify left bottom) hide)
+    )
+    (property "Public" "False" (at 377.19 85.09 0)
+      (effects (font (size 1.27 1.27)) (justify left bottom) hide)
     )
     (pin "1")
@@
       (effects (font (size 1.27 1.27) (thickness 0.15)) (justify left bottom) hide)
     )
+    (property "Public" "False" (at 217.17 187.96 0)
+      (effects (font (size 1.27 1.27)) (justify left bottom) hide)
+    )
     (pin "1")
     (pin "2")
@@
     )
   )
-  (symbol (lib_name "C_100n_0402_3") (lib_id "antmicroCapacitors0402:C_100n_0402") (at 190.5 208.28 90) (unit 1)
+  (symbol (lib_id "antmicroCapacitors0402:C_100n_0402") (at 190.5 208.28 90) (unit 1)
     (in_bom yes) (on_board yes) (dnp no) (fields_autoplaced)
     (property "Reference" "C3" (at 191.135 203.835 90)
@@
       (effects (font (size 1.27 1.27) (thickness 0.15)) (justify left bottom) hide)
     )
+    (property "Public" "False" (at 223.52 187.96 0)
+      (effects (font (size 1.27 1.27)) (justify left bottom) hide)
+    )
     (pin "1")
     (pin "2")
@@
     )
   )
-  (symbol (lib_name "MP_Pad6mm_Drill3mm_2") (lib_id "antmicroMechanicalParts:MP_Pad6mm_Drill3mm") (at 31.75 270.51 0) (unit 1)
+  (symbol (lib_id "antmicroMechanicalParts:MP_Pad6mm_Drill3mm") (at 31.75 270.51 0) (unit 1)
     (in_bom no) (on_board yes) (dnp no)
     (property "Reference" "MP2" (at 40.64 269.24 0)
@@
     )
     (property "Value" "MP_Pad6mm_Drill3mm" (at 40.64 271.78 0)
-      (effects (font (size 1.27 1.27) (thickness 0.15)) (justify left) hide)
+      (effects (font (size 1.27 1.27) (thickness 0.15)) (justify left))
     )
     (property "Footprint" "antmicro-footprints:MP_Pad6mm_Drill3mm" (at 52.07 278.13 0)
@@
     (property "License" "Apache-2.0" (at 52.07 283.21 0)
       (effects (font (size 1.27 1.27) (thickness 0.15)) (justify left bottom) hide)
+    )
+    (property "Public" "False" (at 52.07 285.75 0)
+      (effects (font (size 1.27 1.27)) (justify left bottom) hide)
     )
     (pin "1")
@@
     )
   )
-  (symbol (lib_name "MP_Pad6mm_Drill3mm_1") (lib_id "antmicroMechanicalParts:MP_Pad6mm_Drill3mm") (at 31.75 276.86 0) (unit 1)
+  (symbol (lib_id "antmicroMechanicalParts:MP_Pad6mm_Drill3mm") (at 31.75 276.86 0) (unit 1)
     (in_bom no) (on_board yes) (dnp no)
     (property "Reference" "MP3" (at 40.64 275.59 0)
@@
     )
     (property "Value" "MP_Pad6mm_Drill3mm" (at 40.64 278.13 0)
-      (effects (font (size 1.27 1.27) (thickness 0.15)) (justify left) hide)
+      (effects (font (size 1.27 1.27) (thickness 0.15)) (justify left))
     )
     (property "Footprint" "antmicro-footprints:MP_Pad6mm_Drill3mm" (at 52.07 284.48 0)
@@
     (property "License" "Apache-2.0" (at 52.07 289.56 0)
       (effects (font (size 1.27 1.27) (thickness 0.15)) (justify left bottom) hide)
+    )
+    (property "Public" "False" (at 52.07 292.1 0)
+      (effects (font (size 1.27 1.27)) (justify left bottom) hide)
     )
     (pin "1")
@@
     )
   )
-  (symbol (lib_name "C_100n_0402_2") (lib_id "antmicroCapacitors0402:C_100n_0402") (at 203.2 208.28 90) (unit 1)
+  (symbol (lib_id "antmicroCapacitors0402:C_100n_0402") (at 203.2 208.28 90) (unit 1)
     (in_bom yes) (on_board yes) (dnp no) (fields_autoplaced)
     (property "Reference" "C5" (at 203.835 203.835 90)
@@
       (effects (font (size 1.27 1.27) (thickness 0.15)) (justify left bottom) hide)
     )
+    (property "Public" "False" (at 236.22 187.96 0)
+      (effects (font (size 1.27 1.27)) (justify left bottom) hide)
+    )
     (pin "1")
     (pin "2")
@@
     )
   )
-  (symbol (lib_name "C_10u_0805_35V_1") (lib_id "antmicroCapacitorsmisc:C_10u_0805_35V") (at 283.21 105.41 90) (unit 1)
+  (symbol (lib_id "antmicroCapacitorsmisc:C_10u_0805_35V") (at 283.21 105.41 90) (unit 1)
     (in_bom yes) (on_board yes) (dnp no) (fields_autoplaced)
     (property "Reference" "C1" (at 285.115 101.6 90)
@@
     (property "Author" "Antmicro" (at 308.61 85.09 0)
       (effects (font (size 1.27 1.27) (thickness 0.15)) (justify left bottom) hide)
+    )
+    (property "Public" "False" (at 316.23 85.09 0)
+      (effects (font (size 1.27 1.27)) (justify left bottom) hide)
     )
     (pin "1")
@@
       (effects (font (size 1.27 1.27) (thickness 0.15)) (justify left bottom) hide)
     )
+    (property "Public" "False" (at 398.78 113.03 0)
+      (effects (font (size 1.27 1.27)) (justify left bottom) hide)
+    )
     (pin "1")
     (pin "2")
@@
     )
   )
-  (symbol (lib_name "C_100n_0402_1") (lib_id "antmicroCapacitors0402:C_100n_0402") (at 196.85 208.28 90) (unit 1)
+  (symbol (lib_id "antmicroCapacitors0402:C_100n_0402") (at 196.85 208.28 90) (unit 1)
     (in_bom yes) (on_board yes) (dnp no) (fields_autoplaced)
     (property "Reference" "C4" (at 197.485 203.835 90)
@@
       (effects (font (size 1.27 1.27) (thickness 0.15)) (justify left bottom) hide)
     )
-    (pin "1")
+    (property "Public" "False" (at 229.87 187.96 0)
+      (effects (font (size 1.27 1.27)) (justify left bottom) hide)
+    )
+    (pin "1")
